File: BeerBoard.kicad_pcb (KiCad board)
At the start: 4 copper layers, 45.6 x 94.3 mm, 62 parts, among them J1 Conn_01x10, J2 Conn_01x10, J3 USB_B_Micro, J4 Conn_01x10, J5 Conn_01x10, J6 Conn_02x04_Odd_Even, SW1 SW_BOOT0, SW2 SW_NRST, SW3 SW_SPDT, SW4 SW_NRST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

Commit message: v0.2 - ready for manufactoring
Parts:
- R10, R11, R12, R13, R14, R15, R16, R17, R5, R6, R7, R8, R9: value 100k -> 1k
- R3, R4: value 10k -> 1k
- SW3: value SW_SPDT -> SW_PWR
- moved R11 1.95 mm to (121.1, 104.6)
- moved J3 0.26 mm to (117.8, 98.6), turned to -90 degrees
Connections:
- net I2C_SCL renamed PF6/I2C_SCL
- net I2C_SDA renamed PF7/I2C_SDA
- net PA10 renamed PA10/USART_RX
- net PA4 renamed PA4/SPI_NSS
- net PA5 renamed PA5/SPI_CLOCK
- net PA6 renamed PA6/SPI_MISO
- net PA7 renamed PA7/SPI_MOSI
- net PA9 renamed PA9/USART_TX
Routing:
- net +3.3V: track 11.1 -> 26.4 mm
- net PA1: track 13.9 -> 15.9 mm
- net Net-(D7-A): track 13.0 -> 11.2 mm
- net PB5: track 33.3 -> 32.1 mm
- net BOOT0: track 23.8 -> 24.9 mm
- net PB3: track 32.1 -> 31.1 mm
- net PA3: track 66.9 -> 66.0 mm
- net PB4: track 27.8 -> 27.0 mm
- net PB6: track 38.2 -> 37.5 mm
- net GND: track 23.5 -> 22.9 mm, vias 255 -> 265
- net PB13: track 39.7 -> 39.1 mm
- net PC15: track 23.1 -> 23.7 mm
- removed copper zone on F.Cu, net +3.3V
- removed copper zone on F.Cu, net VBUS

Commit message: version 0.2
Parts:
- J3: footprint USB:AMPHENOL_10118194-0001LF -> Connector_USB:USB_Micro-B_Wuerth_629105150521
- R1, R18, R2: value 100k -> 50k
- R3, R4: value 1k -> 2k4
- moved J3 2.18 mm to (119.9, 98.0)
- moved C3 1.90 mm to (125.1, 95.8), turned to 180 degrees
- moved R11 1.30 mm to (122.3, 104.1), turned to 180 degrees
- moved C11 0.30 mm to (125.0, 93.1)
Routing:
- net Net-(D7-A): track 11.2 -> 10.5 mm
- net GND: track 22.9 -> 23.6 mm, vias 265 -> 256
- net PA1: track 15.9 -> 16.5 mm
- net PC14: track 20.8 -> 21.5 mm
