File: BeerBoard.kicad_sch (KiCad schematic)
At the start: 61 parts, among them J1 Conn_01x10, J2 Conn_01x10, J3 USB_B_Micro, J4 Conn_01x10, J5 Conn_01x10, J6 Conn_02x04_Odd_Even, SW1 SW_BOOT0, SW2 SW_NRST, SW3 SW_PWR, SW4 SW_NRST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

Commit message: v0.2 - ready for manufactoring
Parts:
- R3, R4: value 10k -> 1k
Connections:
- net I2C_SCL renamed PF6/I2C_SCL
- net I2C_SDA renamed PF7/I2C_SDA
- net PA10 renamed PA10/USART_RX
- net PA4 renamed PA4/SPI_NSS
- net PA5 renamed PA5/SPI_CLOCK
- net PA6 renamed PA6/SPI_MISO
- net PA7 renamed PA7/SPI_MOSI
- net PA9 renamed PA9/USART_TX
Other:
- note added: "Buttons (BOOT0, NRST, Extra)"
- note removed: "Buttons (Boot0, NRST, Extra)"
- note removed: "Connectivity"
- moved on the sheet: BT1, C1, C13, C14, C15, C2, D1, D10, D11, D12, D13, D2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

Commit message: version 0.2
Parts:
- J3: footprint USB:AMPHENOL_10118194-0001LF -> Connector_USB:USB_Micro-B_Wuerth_629105150521
- R1, R18, R2: value 100k -> 50k
- R3, R4: value 1k -> 2k4
Other:
- moved on the sheet: J6
Changed lines of the file:
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@@
     (stroke (width 0) (type default))
   )
-  (wire (pts (xy 149.86 156.21) (xy 151.13 156.21))
+  (wire (pts (xy 149.86 160.02) (xy 151.13 160.02))
     (stroke (width 0) (type default))
   )
@@
     (stroke (width 0) (type default))
   )
-  (wire (pts (xy 135.89 156.21) (xy 137.16 156.21))
+  (wire (pts (xy 135.89 160.02) (xy 137.16 160.02))
     (stroke (width 0) (type default))
   )
-  (wire (pts (xy 135.89 153.67) (xy 137.16 153.67))
+  (wire (pts (xy 135.89 157.48) (xy 137.16 157.48))
     (stroke (width 0) (type default))
   )
@@
     (stroke (width 0) (type default))
   )
-  (wire (pts (xy 149.86 153.67) (xy 151.13 153.67))
+  (wire (pts (xy 149.86 157.48) (xy 151.13 157.48))
     (stroke (width 0) (type default))
   )
@@
     (stroke (width 0) (type default))
   )
-  (wire (pts (xy 135.89 147.32) (xy 135.89 148.59))
+  (wire (pts (xy 135.89 151.13) (xy 135.89 152.4))
     (stroke (width 0) (type default))
   )
@@
     (stroke (width 0) (type default))
   )
-  (wire (pts (xy 135.89 157.48) (xy 135.89 156.21))
+  (wire (pts (xy 135.89 161.29) (xy 135.89 160.02))
     (stroke (width 0) (type default))
   )
@@
     (stroke (width 0) (type default))
   )
-  (wire (pts (xy 135.89 151.13) (xy 137.16 151.13))
+  (wire (pts (xy 135.89 154.94) (xy 137.16 154.94))
     (stroke (width 0) (type default))
   )
@@
     (stroke (width 0) (type default))
   )
-  (wire (pts (xy 149.86 151.13) (xy 151.13 151.13))
+  (wire (pts (xy 149.86 154.94) (xy 151.13 154.94))
     (stroke (width 0) (type default))
   )
@@
     (stroke (width 0) (type default))
   )
-  (wire (pts (xy 149.86 148.59) (xy 151.13 148.59))
+  (wire (pts (xy 149.86 152.4) (xy 151.13 152.4))
     (stroke (width 0) (type default))
   )
@@
     (stroke (width 0) (type default))
   )
-  (wire (pts (xy 135.89 148.59) (xy 137.16 148.59))
+  (wire (pts (xy 135.89 152.4) (xy 137.16 152.4))
     (stroke (width 0) (type default))
   )
@@
     )
   )
-  (global_label "PA9{slash}USART_TX" (shape input) (at 135.89 153.67 180) (fields_autoplaced)
+  (global_label "PA9{slash}USART_TX" (shape input) (at 135.89 157.48 180) (fields_autoplaced)
     (effects (font (size 1.27 1.27)) (justify right))
-    (property "Intersheetrefs" "${INTERSHEET_REFS}" (at 118.9953 153.67 0)
+    (property "Intersheetrefs" "${INTERSHEET_REFS}" (at 118.9953 157.48 0)
       (effects (font (size 1.27 1.27)) (justify right) hide)
     )
@@
     )
   )
-  (global_label "PB14" (shape input) (at 151.13 151.13 0) (fields_autoplaced)
+  (global_label "PB14" (shape input) (at 151.13 154.94 0) (fields_autoplaced)
     (effects (font (size 1.27 1.27)) (justify left))
-    (property "Intersheetrefs" "${INTERSHEET_REFS}" (at 159.0742 151.13 0)
+    (property "Intersheetrefs" "${INTERSHEET_REFS}" (at 159.0742 154.94 0)
       (effects (font (size 1.27 1.27)) (justify left) hide)
     )
@@
     )
   )
-  (global_label "PA8" (shape input) (at 151.13 153.67 0) (fields_autoplaced)
+  (global_label "PA8" (shape input) (at 151.13 157.48 0) (fields_autoplaced)
     (effects (font (size 1.27 1.27)) (justify left))
-    (property "Intersheetrefs" "${INTERSHEET_REFS}" (at 157.6833 153.67 0)
+    (property "Intersheetrefs" "${INTERSHEET_REFS}" (at 157.6833 157.48 0)
       (effects (font (size 1.27 1.27)) (justify left) hide)
     )
@@
     )
   )
-  (global_label "PB13" (shape input) (at 151.13 148.59 0) (fields_autoplaced)
+  (global_label "PB13" (shape input) (at 151.13 152.4 0) (fields_autoplaced)
     (effects (font (size 1.27 1.27)) (justify left))
-    (property "Intersheetrefs" "${INTERSHEET_REFS}" (at 159.0742 148.59 0)
+    (property "Intersheetrefs" "${INTERSHEET_REFS}" (at 159.0742 152.4 0)
       (effects (font (size 1.27 1.27)) (justify left) hide)
     )
@@
     )
   )
-  (global_label "PB15" (shape input) (at 135.89 151.13 180) (fields_autoplaced)
+  (global_label "PB15" (shape input) (at 135.89 154.94 180) (fields_autoplaced)
     (effects (font (size 1.27 1.27)) (justify right))
-    (property "Intersheetrefs" "${INTERSHEET_REFS}" (at 127.9458 151.13 0)
+    (property "Intersheetrefs" "${INTERSHEET_REFS}" (at 127.9458 154.94 0)
       (effects (font (size 1.27 1.27)) (justify right) hide)
     )
@@
     )
   )
-  (global_label "PA10{slash}USART_RX" (shape input) (at 151.13 156.21 0) (fields_autoplaced)
+  (global_label "PA10{slash}USART_RX" (shape input) (at 151.13 160.02 0) (fields_autoplaced)
     (effects (font (size 1.27 1.27)) (justify left))
-    (property "Intersheetrefs" "${INTERSHEET_REFS}" (at 169.5366 156.21 0)
+    (property "Intersheetrefs" "${INTERSHEET_REFS}" (at 169.5366 160.02 0)
       (effects (font (size 1.27 1.27)) (justify left) hide)
     )
@@
     )
   )
-  (symbol (lib_id "power:GND") (at 135.89 157.48 0) (unit 1)
+  (symbol (lib_id "power:GND") (at 135.89 161.29 0) (unit 1)
     (in_bom yes) (on_board yes) (dnp no) (fields_autoplaced)
-    (property "Reference" "#PWR020" (at 135.89 163.83 0)
+    (property "Reference" "#PWR020" (at 135.89 167.64 0)
       (effects (font (size 1.27 1.27)) hide)
     )
-    (property "Value" "GND" (at 135.89 162.56 0)
+    (property "Value" "GND" (at 135.89 166.37 0)
       (effects (font (size 1.27 1.27)))
     )
-    (property "Footprint" "" (at 135.89 157.48 0)
+    (property "Footprint" "" (at 135.89 161.29 0)
       (effects (font (size 1.27 1.27)) hide)
     )
-    (property "Datasheet" "" (at 135.89 157.48 0)
+    (property "Datasheet" "" (at 135.89 161.29 0)
       (effects (font (size 1.27 1.27)) hide)
     )
@@
       (effects (font (size 1.27 1.27)) (justify right))
     )
-    (property "Value" "100k" (at 214.63 44.45 0)
+    (property "Value" "50k" (at 214.63 44.45 0)
       (effects (font (size 1.27 1.27)) (justify right))
     )
@@
       (effects (font (size 1.27 1.27)) (justify right))
     )
-    (property "Value" "100k" (at 247.65 44.45 0)
+    (property "Value" "50k" (at 247.65 44.45 0)
       (effects (font (size 1.27 1.27)) (justify right))
     )
@@
     )
   )
-  (symbol (lib_id "Connector_Generic:Conn_02x04_Odd_Even") (at 142.24 151.13 0) (unit 1)
+  (symbol (lib_id "Connector_Generic:Conn_02x04_Odd_Even") (at 142.24 154.94 0) (unit 1)
     (in_bom yes) (on_board yes) (dnp no)
-    (property "Reference" "J6" (at 143.51 144.78 0)
+    (property "Reference" "J6" (at 143.51 148.59 0)
       (effects (font (size 1.27 1.27)))
     )
-    (property "Value" "Conn_02x04_Odd_Even" (at 143.51 144.78 0)
+    (property "Value" "Conn_02x04_Odd_Even" (at 143.51 148.59 0)
       (effects (font (size 1.27 1.27)) hide)
     )
-    (property "Footprint" "Connector_PinHeader_2.54mm:PinHeader_2x04_P2.54mm_Vertical" (at 142.24 151.13 0)
+    (property "Footprint" "Connector_PinHeader_2.54mm:PinHeader_2x04_P2.54mm_Vertical" (at 142.24 154.94 0)
       (effects (font (size 1.27 1.27)) hide)
     )
-    (property "Datasheet" "~" (at 142.24 151.13 0)
+    (property "Datasheet" "~" (at 142.24 154.94 0)
       (effects (font (size 1.27 1.27)) hide)
     )
@@
       (effects (font (size 1.27 1.27)) (justify right))
     )
-    (property "Value" "1k" (at 25.4 160.02 0)
+    (property "Value" "2k4" (at 25.4 160.02 0)
       (effects (font (size 1.27 1.27)) (justify right))
     )
@@
       (effects (font (size 1.27 1.27)) (justify right))
     )
-    (property "Value" "1k" (at 34.29 160.02 0)
+    (property "Value" "2k4" (at 34.29 160.02 0)
       (effects (font (size 1.27 1.27)) (justify right))
     )
@@
       (effects (font (size 1.27 1.27)))
     )
-    (property "Footprint" "USB:AMPHENOL_10118194-0001LF" (at 34.29 40.64 0)
+    (property "Footprint" "Connector_USB:USB_Micro-B_Wuerth_629105150521" (at 34.29 40.64 0)
       (effects (font (size 1.27 1.27)) hide)
     )
@@
     )
   )
-  (symbol (lib_id "power:VDD") (at 135.89 147.32 0) (unit 1)
+  (symbol (lib_id "power:VDD") (at 135.89 151.13 0) (unit 1)
     (in_bom yes) (on_board yes) (dnp no) (fields_autoplaced)
-    (property "Reference" "#PWR034" (at 135.89 151.13 0)
+    (property "Reference" "#PWR034" (at 135.89 154.94 0)
       (effects (font (size 1.27 1.27)) hide)
     )
-    (property "Value" "VDD" (at 135.89 142.24 0)
+    (property "Value" "VDD" (at 135.89 146.05 0)
       (effects (font (size 1.27 1.27)))
     )
-    (property "Footprint" "" (at 135.89 147.32 0)
+    (property "Footprint" "" (at 135.89 151.13 0)
       (effects (font (size 1.27 1.27)) hide)
     )
-    (property "Datasheet" "" (at 135.89 147.32 0)
+    (property "Datasheet" "" (at 135.89 151.13 0)
       (effects (font (size 1.27 1.27)) hide)
     )
@@
       (effects (font (size 1.27 1.27)) (justify right))
     )
-    (property "Value" "100k" (at 182.88 57.15 0)
+    (property "Value" "50k" (at 182.88 57.15 0)
       (effects (font (size 1.27 1.27)) (justify right))
     )
